File: projects/valvestudio/benchpowersupply/vsBenchPowerSupply.sch (EAGLE design)
At the start: 42 parts, among them Q1 STN1HNK60, Q3 BC337

Commit message: added more examples to notebook cleaned up some formatting
Parts:
- removed D6: (no value), holla:LED-3MM-0.1
- removed J10: (no value), holla:SWITCH-PANEL-DPDT
- removed J11: (no value), holla:CONN-04-3.81MM-PLUGIN-SCREW
- removed J6, J8: (no value), holla:CONN-02-3.81MM-PLUGIN-SCREW
- removed J7, J9: (no value), holla:CONN-03-3.81MM-PLUGIN-SCREW
- removed T1: (no value), holla:TRANSFORMER-3-2
- removed T2: (no value), holla:TRANSFORMER-2-2
- added BF1, BF2, BIASOUT+, BIASOUT-, F12.6A, F12.6B, F12.6CT, F5A, F5B, F5CT, F6.3A, F6.3B, F6.3CT, GND, LINE, LINEVAR, NEUTRAL, PA, PB, PF1, PF2, PLATEOUT+, PLATEOUT-, PRECT, SA, SB, SCREENOUT+, SCREENOUT-, SF1, SF2, SRECT: (no value), holla:TESTPOINTTHRU
- added C10, C2, C3, C4, C5, C6, C7, C8: (no value), holla:C-POLARIZED-SMD-E-3MM
- added F3, F4, F5, F6: (no value), holla:FUSE-HOLDER-3557-2
- added GL1, GL2, GL3, GL4, GL5: (no value), holla:INDICATOR-NEON-BULB-NE2-DRILL
- added L1, L2: (no value), holla:INDUCTOR-0805
- added M10, M5, M7: (no value), holla:METER-PANEL-ANALOG-CURRENT-PLUGIN-3.81MM
- added M6, M8, M9: (no value), holla:METER-PANEL-ANALOG-VOLTAGE-PLUGIN-3.81MM
- added R10, R11, R12, R13, R14, R15, R16, R17: (no value), holla:R-0402
- added R19, R20: (no value), holla:POTENTIOMETER
- added S10, S11, S12, S13, S14, S15, S2, S3, S4, S5, S6, S7, S8, S9: (no value), holla:SWITCH-PANEL-SPST
- added T100, T1000, T12.6, T5.0, T6.3, T600: (no value), holla:TRANSFORMER-3-2
- added T120: (no value), holla:TRANSFORMER-2-2
- added U$2, U$3: OUTLET-RECEPTACLE, holla:OUTLET-RECEPTACLE
- J3: device holla:CONN-03-3.81MM-PLUGIN-SCREW -> holla:OUTLET-RECEPTABLE-SINGLE
- J4: device holla:CONN-02-3.81MM-PLUGIN-SCREW -> holla:OUTLET-RECEPTABLE-SINGLE
- J5: device holla:CONN-02-.156 -> holla:OUTLET-RECEPTABLE-SINGLE
- R9: device holla:R-0805 -> holla:R-0402
- U$1: value OUTLET-RECEPTABLE -> OUTLET-RECEPTACLE; device holla:OUTLET-RECEPTABLE -> holla:OUTLET-RECEPTACLE
Connections:
- removed net HVA: J10.S1, T1.P1
- removed net HVB: J10.S2, T1.P2
- removed net HVCT: T1.PCT
- removed net HVRECT: D4.C, D5.C, J11.1, T2.S1
- removed net VFIL5: J11.2, T2.S2
- new net BIASOUT: BIASOUT+.P$1, M10.-, M9.-
- new net BIASOUT-: BIASOUT-.P$1, C10.+, C7.+, M9.+, R20.1, T100.PCT
- new net F6.3B: F6.3B.P$1, T6.3.P1
- new net HVOUT: M5.-, M6.+, PLATEOUT+.P$1
- new net LINE: F3.P$1, F4.P$1, F5.P$1, F6.P$1, J3.LINE, LINE.P$1, M3.-, R8.2, U$1.LINE, U$2.LINE, U$3.LINE
- new net LINEVAR: J5.LINE, LINEVAR.P$1, M4.+, R8.W, T120.P1
- new net N$17: GL1.A, S2.2, T1000.S1
- new net N$30: J4.LINE, T120.S1
- new net N$31: BF2.P$1, C7.-, R15.1, R20.2
- new net N$32: L2.P$1, M7.+, R16.1, S11.2, S12.1, SF2.P$1
- new net N$33: M10.+, R20.W
- new net N$34: BF1.P$1, C10.-, D4.A, D5.A, R15.2
- new net N$35: J4.NEU, T120.S2
- new net N$36: F5.P$2, S14.1
- new net N$37: GL4.A, S14.2, T100.S1
- new net N$39: F4.P$2, S13.1
- new net N$41: F3.P$2, S15.1
- new net N$44: F6.P$2, S2.1
- new net NEUTRAL: GL1.A1, GL2.A1, GL3.A1, GL4.A1, GL5.A1, J12.2, J3.NEU, J5.NEU, M4.-, NEUTRAL.P$1, R19.1, R8.1, T100.S2, T1000.S2, T12.6.S2, T120.P2, T5.0.S2, T6.3.S2, T600.S2, U$1.NEU, U$2.NEU, U$3.NEU
- new net PA: PA.P$1, T1000.P1
- new net PB: PB.P$1, T1000.P2
- new net PLATECT: C3.-, C5.-, M6.-, PLATEOUT-.P$1, R11.1, R14.1, T1000.PCT
- new net PRECT: PF1.P$1, PRECT.P$1, S3.1, S4.1, S5.1, S6.1
- new net SA: SA.P$1, T600.P1
- new net SB: SB.P$1, T600.P2
- new net SCREENCT: C6.-, C8.-, M8.-, R17.1, R9.1, SCREENOUT-.P$1, T600.PCT
- new net SCREENOUT: M7.-, M8.+, SCREENOUT+.P$1
- new net SRECT: S10.1, S11.1, S8.1, S9.1, SF1.P$1, SRECT.P$1
- new net VFIL12A: F12.6A.P$1, T12.6.P2
- new net VFIL12B: F12.6B.P$1, T12.6.P1
- new net VFIL12CT: F12.6CT.P$1, T12.6.PCT
- new net VFIL5A: F5A.P$1, T5.0.P2
- new net VFIL5B: F5B.P$1, T5.0.P1
- new net VFIL5CT: F5CT.P$1, T5.0.PCT
- new net VFIL6A: F6.3A.P$1, T6.3.P2
- new net VFIL6CT: F6.3CT.P$1, T6.3.PCT
- net GND: now also GND.P$1, J3.GND, J4.GND, J5.GND, U$2.GND, U$3.GND; no longer J3.1
- net N$10: now also C2.+, R10.2, S3.2; no longer J3.3, J4.1
- net N$11: now also L1.P$1, M5.+, PF2.P$1, R12.1, S6.2, S7.1; no longer J4.2, J7.1
- net N$12: now also C2.-, C3.+, R10.1, R11.2; no longer J3.2, J5.2, J7.2, J8.2
- net N$13: now also L1.P$2, S4.2; no longer J6.1, J7.3
- net N$14: now also R12.2, S5.2; no longer J5.1, J6.2
- net N$15: now also R19.W, T600.S1; no longer D4.A, J10.S1A
- net N$16: now also C4.+, R13.2, S7.2; no longer J10.S1B, J11.4
- net N$18: now also C4.-, C5.+, R13.1, R14.2; no longer J8.1
- net N$20: now also GL3.A, R19.2, S13.2; no longer J9.1
- net N$21: now also C6.+, R9.2, S8.2; no longer J9.3
- net N$23: now also GL5.A, S15.2, T12.6.S1, T5.0.S1, T6.3.S1; no longer D6.A, R8.2, S1.2, T2.P1
- net N$24: now also GL2.A, M3.+, S1.2; no longer J12.2, M4.-, R8.1, R9.1, T1.S2, T2.P2, U$1.NEU
- net N$25: now also L2.P$2, S9.2; no longer D6.C, R9.2
- net N$26: now also D4.C, T100.P1; no longer M3.+, R8.W
- net N$27: now also D5.C, T100.P2; no longer M3.-, M4.+, T1.S1, U$1.LINE
- net N$28: now also R16.2, S10.2; no longer D5.A, J10.S2A
- net N$29: now also C8.+, R17.2, S12.2; no longer J10.S2B, J11.3
Other:
- note added: "100V"
- note added: "12.6VAC"
- note added: "130VAC"
- note added: "1A"
- note added: "300V"
- note added: "50mA"
- note added: "50uA"
- note added: "5A"
- note added: "6.3VAC"
- note added: "750V"
- note added: "BIAS ENABLE"
- note added: "FILAMENT ENABLE"
- note added: "FRONT"
- note added: "ISOLATED"
- note added: "NEUT"
- note added: "PLATE ENABLE"
- note added: "POWER"
- note added: "REAR"
- note added: "RECTIFIER PLUGIN"
- note added: "SCREEN ENABLE"
- note added: "VSPS FILAMENT 5.0VAC-CT@4A FILAMENT 6.3VAC-CT@3A FILAMENT 12.6VAC-CT@3A GRID -100DC@10mA Variable SCREEN 600VAC-CT@50mA Variable PLATE 1000VAC-CT@500mA Variable"
- note added: "http://www.jameco.com/z/R9-71N-05-120V-RED-R-Lamp-Panel-Red-Neon-120VoltSolder-Terminals-W-Bulb_215803.html"
- note removed: "AC Ammeter"
- note removed: "AC Voltmeter"
- note removed: "FUSE"
- note removed: "NEUTRAL"
- note removed: "change foot print of rectifier diodes"
- moved on the sheet: D4, D5, F2, J12, R8, R9
