File: projects/valvestudio/benchpowersupply/schematic/vsBenchPowerSupply.brd (EAGLE design)
At the start: 160 x 100 mm, 122 parts, among them Q1 STN1HNK60, Q3 BC337

Commit message: initial add for most
Parts:
- added GND19, GND21, GND23, GND25, PF3, PF4, SF3, SF4: (no value), holla:TPTHRU
- added J10, J11, J13, J9: (no value), holla:CONN-3.81MM-KF2EDG-3
- added J6, J7, J8: (no value), holla:CONN-.100-2
- added U$4: OUTLET-RECEPTACLE, holla:CONN-3.81MM-KF2EDG-3
Connections:
- new net N$38: F3.1@1, F3.1@2, J9.3
- new net N$40: F6.1@1, F6.1@2, J10.3
- new net N$42: F4.1@1, F4.1@2, J11.3
- new net N$43: F5.1@1, F5.1@2, J13.3
- net GND: now also GND19.1, GND21.1, GND23.1, GND25.1, J10.1, J11.1, J13.1, J9.1, U$4.1
- net LINE: no longer F3.1@1, F3.1@2, F4.1@1, F4.1@2, F5.1@1, F5.1@2, F6.1@1, F6.1@2
- net LINEVAR: now also J6.1, U$4.3
- net N$11: now also PF4.1
- net N$32: now also SF4.1
- net NEUTRAL: now also J10.2, J11.2, J13.2, J6.2, J9.2, U$4.2
- net PLATECT: now also J7.2
- net PRECT: now also J7.1, PF3.1
- net SCREENCT: now also J8.2
- net SRECT: now also J8.1, SF3.1

Commit message: big submit, should do this more often, duh!
Parts:
- removed R19, R8: (no value), holla:CONN-.100-3
- added BF3, BF4, BF5, BF6, F6.3A1, F6.3A2, F6.3B1, F6.3B2, GGND, PF5, PFA, PFB, PGND, SFA, SFB, SGND: (no value), holla:TPTHRU
- added C11, C9: (no value), holla:E-3
- added D6, D7: (no value), holla:DO-35
- added J14, S16, S17, S18, S19, S20: (no value), holla:CONN-.100-2
- added J15, J16, J17: (no value), holla:CONN-.100-3
- added J18: (no value), holla:CONN-3.81MM-KF2EDG-3
- added R18, R21, R23, R24, R25: (no value), holla:R0402
- added T1, T2: (no value), holla:TRANSFORMER-4-2-G
- renumbered BIASOUT+ to GRIDOUT+, BIASOUT- to GRIDOUT-
Connections:
- removed net BIASOUT-: C10.+, C7.+, GRIDOUT-.1, M9.2, R20.1, T100.4
- new net N$42: BF3.1, C10.-, D4.A, D5.A, R18.2
- new net N$45: J16.2, T1000.1
- new net N$46: J17.3, S16.2
- new net N$47: PFB.1, T1.5
- new net N$48: PFA.1, T1.6
- new net N$49: J16.3, S19.2
- new net N$50: R20.2
- new net N$51: M10.1, S18.1
- new net N$52: SFB.1, T2.5
- new net N$53: SFA.1, T2.6
- new net N$55: BF4.1, C7.-, R18.1, R20.1, R25.1
- new net N$56: C10.+, C11.-, C7.+, C9.-, GRIDOUT-.1, M9.2, R24.1, R25.2, T100.4
- new net N$57: D4.C, D6.A, T100.3
- new net N$58: R23.1, S20.1
- net BIASOUT: now also BF6.1, S17.2, S18.2, S20.2; no longer M10.1
- net GND: now also GGND.1, J18.1, PGND.1, SGND.1
- net LINE: now also J15.3, J18.3; no longer R8.3
- net LINEVAR: now also J15.2; no longer R8.2
- net N$15: now also J17.2; no longer R19.2
- net N$17: now also S19.1, T1.1; no longer T1000.1
- net N$20: now also S16.1, T2.1; no longer R19.3
- net N$26: now also BF5.1, M10.2, R21.2, R23.2; no longer D4.C, T100.3
- net N$27: now also D7.A
- net N$31: now also C11.+, R24.2; no longer C7.-
- net N$33: now also R21.1, S17.1; no longer M10.2, R20.2
- net N$34: now also C9.+, D6.C, D7.C; no longer C10.-, D4.A, D5.A
- net NEUTRAL: now also J15.1, J16.1, J17.1, J18.2, T1.2, T2.2; no longer R19.1, R8.1
