File: projects/valvestudio/benchpowersupply/schematic/vsBenchPowerSupply.sch (EAGLE design)
At the start: 122 parts, among them Q1 STN1HNK60, Q3 BC337

Commit message: added some labels
Other:
- note added: "HAVE"
- note added: "WIND"
Changed lines of the file:
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@@
 <wire x1="136.398" y1="194.056" x2="144.018" y2="194.056" width="0.1524" layer="97"/>
 <text x="66.548" y="194.056" size="1.778" layer="97" ratio="15">FRONT</text>
+<text x="131.572" y="174.752" size="1.778" layer="97">HAVE</text>
+<text x="134.366" y="129.286" size="1.778" layer="97">HAVE</text>
+<text x="45.72" y="12.7" size="1.778" layer="97">WIND</text>
+<text x="58.674" y="123.444" size="1.778" layer="97">WIND</text>
+<text x="50.8" y="68.58" size="1.778" layer="97">WIND</text>
 </plain>
 <instances>

Commit message: initial add for most
Parts:
- added GND19, GND21, GND23, GND25, PF3, PF4, SF3, SF4: (no value), holla:TESTPOINTTHRU
- added J10, J11, J13, J9: (no value), holla:CONN-03-3.81MM-PLUGIN-SCREW
- added J6, J7, J8: (no value), holla:METER-PANEL-HV-WARNING
- added U$4: OUTLET-RECEPTACLE, holla:OUTLET-RECEPTACLE
Connections:
- new net N$38: F3.P$1, J9.3
- new net N$40: F6.P$1, J10.3
- new net N$42: F4.P$1, J11.3
- new net N$43: F5.P$1, J13.3
- net GND: now also GND19.P$1, GND21.P$1, GND23.P$1, GND25.P$1, J10.1, J11.1, J13.1, J9.1, U$4.GND
- net LINE: no longer F3.P$1, F4.P$1, F5.P$1, F6.P$1
- net LINEVAR: now also J6.P$1, U$4.LINE
- net N$11: now also PF4.P$1
- net N$32: now also SF4.P$1
- net NEUTRAL: now also J10.2, J11.2, J13.2, J6.P$2, J9.2, U$4.NEU
- net PLATECT: now also J7.P$2
- net PRECT: now also J7.P$1, PF3.P$1
- net SCREENCT: now also J8.P$2
- net SRECT: now also J8.P$1, SF3.P$1
Other:
- note added: "FILAMENT SUPPLY"
- note added: "GRID SUPPLY"
- note added: "LINEVAR"
- note added: "MAINS"
- note added: "PLATE SUPPLY"
- note added: "SCREEN SUPPLY"
- note added: "VSPS FILAMENT 5.0VAC-CT@6A FILAMENT 6.3VAC-CT@6A FILAMENT 12.6VAC-CT@4A GRID -100VDC@10mA Variable SCREEN 400VDC@100mA Variable PLATE 550VDC@500mA Variable"
- note added: "may need to be larger"
- note added: "rotary?"
- note removed: "300V"
- note removed: "50mA"
- note removed: "VSPS FILAMENT 5.0VAC-CT@4A FILAMENT 6.3VAC-CT@3A FILAMENT 12.6VAC-CT@3A GRID -100DC@10mA Variable SCREEN 600VAC-CT@50mA Variable PLATE 1000VAC-CT@500mA Variable"

Commit message: big submit, should do this more often, duh!
Parts:
- removed BIASOUT+, BIASOUT-: (no value), holla:TESTPOINTTHRU
- removed R19, R8: (no value), holla:POTENTIOMETER
- added BF3, BF4, BF5, BF6, F6.3A1, F6.3A2, F6.3B1, F6.3B2, GGND, GRIDOUT+, GRIDOUT-, PF5, PFA, PFB, PGND, SFA, SFB, SGND: (no value), holla:TESTPOINTTHRU
- added C11, C9: (no value), holla:C-POLARIZED-SMD-E-3MM
- added D6, D7: (no value), holla:DIODE-1N4148
- added J14: (no value), holla:METER-PANEL-HV-WARNING
- added J15, J16, J17: (no value), holla:VARIAC
- added J18: (no value), holla:OUTLET-RECEPTABLE-SINGLE
- added R18, R21, R23, R24, R25: (no value), holla:R-0402
- added S16, S17, S18, S19, S20: (no value), holla:SWITCH-PANEL-SPST
- added T1, T2: (no value), holla:TRANSFORMER-2-2
Connections:
- removed net BIASOUT-: BIASOUT-.P$1, C10.+, C7.+, M9.+, R20.1, T100.PCT
- new net N$42: BF3.P$1, C10.-, D4.A, D5.A, R18.2
- new net N$45: J16.W, T1000.S1
- new net N$46: J17.2, S16.2
- new net N$47: PFB.P$1, T1.S1
- new net N$48: PFA.P$1, T1.S2
- new net N$49: J16.2, S19.2
- new net N$50: R20.W
- new net N$51: M10.-, S18.1
- new net N$52: SFB.P$1, T2.S1
- new net N$53: SFA.P$1, T2.S2
- new net N$55: BF4.P$1, C7.-, R18.1, R20.1, R25.1
- new net N$56: C10.+, C11.-, C7.+, C9.-, GRIDOUT-.P$1, M9.+, R24.1, R25.2, T100.PCT
- new net N$57: D4.C, D6.A, T100.P1
- new net N$58: R23.1, S20.1
- net BIASOUT: now also BF6.P$1, GRIDOUT+.P$1, S17.2, S18.2, S20.2; no longer BIASOUT+.P$1, M10.-
- net GND: now also GGND.P$1, J18.GND, PGND.P$1, SGND.P$1
- net LINE: now also J15.2, J18.LINE; no longer R8.2
- net LINEVAR: now also J15.W; no longer R8.W
- net N$15: now also J17.W; no longer R19.W
- net N$17: now also S19.1, T1.P1; no longer T1000.S1
- net N$20: now also S16.1, T2.P1; no longer R19.2
- net N$26: now also BF5.P$1, M10.+, R21.2, R23.2; no longer D4.C, T100.P1
- net N$27: now also D7.A
- net N$31: now also C11.+, R24.2; no longer C7.-
- net N$33: now also R21.1, S17.1; no longer M10.+, R20.W
- net N$34: now also C9.+, D6.C, D7.C; no longer C10.-, D4.A, D5.A
- net NEUTRAL: now also J15.1, J16.1, J17.1, J18.NEU, T1.P2, T2.P2; no longer R19.1, R8.1
Other:
- note added: "+/-100uA"
- note added: "+/-50V"
- note added: "+12.6VDC"
- note added: "+6.3VDC"
- note added: "300mA"
- note added: "500mA"
- note added: "750VDC"
- note added: "All test points on front panel"
- note added: "HV Warning"
- note added: "VSPS FILAMENT 5.0VAC-CT@6A FILAMENT 6.3VAC-CT@6A FILAMENT 12.6VAC-CT@5A GRID +/-50VDC@50mA Variable SCREEN 400VDC@100mA Variable PLATE 550VDC@500mA Variable"
- note added: "probably want PP transistor here."
- note removed: "100V"
- note removed: "1A"
- note removed: "50uA"
- note removed: "LINEVAR"
- note removed: "VSPS FILAMENT 5.0VAC-CT@6A FILAMENT 6.3VAC-CT@6A FILAMENT 12.6VAC-CT@4A GRID -100VDC@10mA Variable SCREEN 400VDC@100mA Variable PLATE 550VDC@500mA Variable"
- note removed: "may need to be larger"
- moved on the sheet: BF1, BF2, C10, C2, C3, C4, C5, C6, C7, C8, D4, D5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

Commit message: initial add for most little tweaks for rest
Other:
- note added: "A"
- note added: "ADC"
- note added: "ADJ"
- note added: "AMP"
- note added: "BATT"
- note added: "CHRG"
- note added: "CPU WiFi"
- note added: "DAC"
- note added: "DISP"
- note added: "ENABLE"
- note added: "ESTOP"
- note added: "HV DC PS 400V@800mA"
- note added: "ISENSE"
- note added: "OUT"
- note added: "RPI3"
- note added: "V"
- note added: "VAR"
- note added: "WARN"

Commit message: initial add
Other:
- note added: "ADC0"
- note added: "ADC1"
- note added: "ADC2"
- note added: "ADC3"
- note added: "DAC0"
- note added: "PGA"
- note added: "PS"
- note added: "SCALE"
- note added: "panel"
- note removed: "ADC"
- note removed: "BATT"
- note removed: "CHRG"
- note removed: "DAC"
